File: _autosave-Magma_STLink.sch (KiCad schematic (older format))
At the start: 44 parts

Commit message: STLink şematikleri değiştirildi. Konnektörlerin kararlaştırılması gerekiyor. PCB boyutu önemli. USB ESD koruması eklendi.SWDIO ve SWCLK pinlerine tekli koruma diyotu eklendi.
Parts:
- R?: footprint (none) -> Resistor_SMD:R_0805_2012Metric_Pad1.20x1.40mm_HandSolder
- U?: footprint (none) -> Package_TO_SOT_SMD:SOT-223-3_TabPin2
Changed lines of the file:
@@
 Connection ~ 4500 1950
 $Comp
-L power:+3.3V #PWR?
+L power:+3.3V #PWR0101
 U 1 1 6148A7FB
 P 4600 1500
-F 0 "#PWR?" H 4600 1350 50  0001 C CNN
+F 0 "#PWR0101" H 4600 1350 50  0001 C CNN
 F 1 "+3.3V" H 4615 1673 50  0000 C CNN
 F 2 "" H 4600 1500 50  0001 C CNN
@@
 UART_RX
 $Comp
-L power:+3.3V #PWR?
+L power:+3.3V #PWR0102
 U 1 1 6148DC33
 P 6250 1550
-F 0 "#PWR?" H 6250 1400 50  0001 C CNN
+F 0 "#PWR0102" H 6250 1400 50  0001 C CNN
 F 1 "+3.3V" H 6265 1723 50  0000 C CNN
 F 2 "" H 6250 1550 50  0001 C CNN
@@
 	5450 3450 5800 3450
 $Comp
-L power:GND #PWR?
+L power:GND #PWR0103
 U 1 1 61494807
 P 5800 3500
-F 0 "#PWR?" H 5800 3250 50  0001 C CNN
+F 0 "#PWR0103" H 5800 3250 50  0001 C CNN
 F 1 "GND" H 5805 3327 50  0000 C CNN
 F 2 "" H 5800 3500 50  0001 C CNN
@@
 $EndComp
 $Comp
-L power:+3.3V #PWR?
+L power:+3.3V #PWR0104
 U 1 1 61495A4A
 P 5450 2950
-F 0 "#PWR?" H 5450 2800 50  0001 C CNN
+F 0 "#PWR0104" H 5450 2800 50  0001 C CNN
 F 1 "+3.3V" H 5465 3123 50  0000 C CNN
 F 2 "" H 5450 2950 50  0001 C CNN
@@
 $EndComp
 $Comp
-L power:GND #PWR?
+L power:GND #PWR0105
 U 1 1 614A0D5A
 P 4600 5350
-F 0 "#PWR?" H 4600 5100 50  0001 C CNN
+F 0 "#PWR0105" H 4600 5100 50  0001 C CNN
 F 1 "GND" H 4605 5177 50  0000 C CNN
 F 2 "" H 4600 5350 50  0001 C CNN
@@
 	8550 2100 8600 2100
 $Comp
-L power:GND #PWR?
+L power:GND #PWR0106
 U 1 1 614A94F9
 P 8600 2200
-F 0 "#PWR?" H 8600 1950 50  0001 C CNN
+F 0 "#PWR0106" H 8600 1950 50  0001 C CNN
 F 1 "GND" H 8605 2027 50  0000 C CNN
 F 2 "" H 8600 2200 50  0001 C CNN
@@
 F 0 "U?" H 1900 1492 50  0000 C CNN
 F 1 "LM1117-3.3" H 1900 1401 50  0000 C CNN
-F 2 "" H 1900 1250 50  0001 C CNN
+F 2 "Package_TO_SOT_SMD:SOT-223-3_TabPin2" H 1900 1250 50  0001 C CNN
 F 3 "http://www.ti.com/lit/ds/symlink/lm1117.pdf" H 1900 1250 50  0001 C CNN
 	1    1900 1250
@@
 $EndComp
 $Comp
-L power:VBUS #PWR?
+L power:VBUS #PWR0107
 U 1 1 614B3CD8
 P 9400 1150
-F 0 "#PWR?" H 9400 1000 50  0001 C CNN
+F 0 "#PWR0107" H 9400 1000 50  0001 C CNN
 F 1 "VBUS" H 9415 1323 50  0000 C CNN
 F 2 "" H 9400 1150 50  0001 C CNN
@@
 $EndComp
 $Comp
-L power:VBUS #PWR?
+L power:VBUS #PWR0108
 U 1 1 614B92E9
 P 1050 800
-F 0 "#PWR?" H 1050 650 50  0001 C CNN
+F 0 "#PWR0108" H 1050 650 50  0001 C CNN
 F 1 "VBUS" H 1065 973 50  0000 C CNN
 F 2 "" H 1050 800 50  0001 C CNN
@@
 	1050 1250 1350 1250
 $Comp
-L power:GND #PWR?
+L power:GND #PWR0109
 U 1 1 614BED35
 P 1900 1700
-F 0 "#PWR?" H 1900 1450 50  0001 C CNN
+F 0 "#PWR0109" H 1900 1450 50  0001 C CNN
 F 1 "GND" H 1905 1527 50  0000 C CNN
 F 2 "" H 1900 1700 50  0001 C CNN
@@
 Connection ~ 2350 1700
 $Comp
-L power:+3.3V #PWR?
+L power:+3.3V #PWR0110
 U 1 1 614CE8FE
 P 2650 1150
-F 0 "#PWR?" H 2650 1000 50  0001 C CNN
+F 0 "#PWR0110" H 2650 1000 50  0001 C CNN
 F 1 "+3.3V" H 2665 1323 50  0000 C CNN
 F 2 "" H 2650 1150 50  0001 C CNN
@@
 Connection ~ 6750 2100
 $Comp
-L power:GND #PWR?
+L power:GND #PWR0111
 U 1 1 614F0B7D
 P 6350 2250
-F 0 "#PWR?" H 6350 2000 50  0001 C CNN
+F 0 "#PWR0111" H 6350 2000 50  0001 C CNN
 F 1 "GND" H 6355 2077 50  0000 C CNN
 F 2 "" H 6350 2250 50  0001 C CNN
@@
 $EndComp
 $Comp
-L power:+3V3 #PWR?
+L power:+3V3 #PWR0112
 U 1 1 614F52DC
 P 10150 1150
-F 0 "#PWR?" H 10150 1000 50  0001 C CNN
+F 0 "#PWR0112" H 10150 1000 50  0001 C CNN
 F 1 "+3V3" H 10165 1323 50  0000 C CNN
 F 2 "" H 10150 1150 50  0001 C CNN
@@
 	3400 4650 3900 4650
 $Comp
-L power:GND #PWR?
+L power:GND #PWR0113
 U 1 1 61540056
 P 3150 2400
-F 0 "#PWR?" H 3150 2150 50  0001 C CNN
+F 0 "#PWR0113" H 3150 2150 50  0001 C CNN
 F 1 "GND" H 3155 2227 50  0000 C CNN
 F 2 "" H 3150 2400 50  0001 C CNN
@@
 	800  3200 1150 3200
 $Comp
-L power:+3V3 #PWR?
+L power:+3V3 #PWR0114
 U 1 1 6155E309
 P 750 2400
-F 0 "#PWR?" H 750 2250 50  0001 C CNN
+F 0 "#PWR0114" H 750 2250 50  0001 C CNN
 F 1 "+3V3" H 765 2573 50  0000 C CNN
 F 2 "" H 750 2400 50  0001 C CNN
@@
 $EndComp
 $Comp
-L power:GND #PWR?
+L power:GND #PWR0115
 U 1 1 61563B99
 P 700 3500
-F 0 "#PWR?" H 700 3250 50  0001 C CNN
+F 0 "#PWR0115" H 700 3250 50  0001 C CNN
 F 1 "GND" H 705 3327 50  0000 C CNN
 F 2 "" H 700 3500 50  0001 C CNN
@@
 Connection ~ 3150 2150
 $Comp
-L power:+3.3V #PWR?
+L power:+3.3V #PWR0116
 U 1 1 61573ADB
 P 2500 2050
-F 0 "#PWR?" H 2500 1900 50  0001 C CNN
+F 0 "#PWR0116" H 2500 1900 50  0001 C CNN
 F 1 "+3.3V" H 2515 2223 50  0000 C CNN
 F 2 "" H 2500 2050 50  0001 C CNN
@@
 	9800 3950 9900 3950
 $Comp
-L power:GND #PWR?
+L power:GND #PWR0117
 U 1 1 614B11D3
 P 10600 3950
-F 0 "#PWR?" H 10600 3700 50  0001 C CNN
+F 0 "#PWR0117" H 10600 3700 50  0001 C CNN
 F 1 "GND" V 10605 3822 50  0000 R CNN
 F 2 "" H 10600 3950 50  0001 C CNN
@@
 	10200 3950 10600 3950
 $Comp
-L power:+3V3 #PWR?
+L power:+3V3 #PWR0118
 U 1 1 614CF9A9
 P 10600 4300
-F 0 "#PWR?" H 10600 4150 50  0001 C CNN
+F 0 "#PWR0118" H 10600 4150 50  0001 C CNN
 F 1 "+3V3" V 10615 4428 50  0000 L CNN
 F 2 "" H 10600 4300 50  0001 C CNN
@@
 	6600 4950 7000 4950
 $Comp
-L power:GND #PWR?
+L power:GND #PWR0119
 U 1 1 614DFCBB
 P 6650 5050
-F 0 "#PWR?" H 6650 4800 50  0001 C CNN
+F 0 "#PWR0119" H 6650 4800 50  0001 C CNN
 F 1 "GND" V 6655 4922 50  0000 R CNN
 F 2 "" H 6650 5050 50  0001 C CNN
@@
 $EndComp
 $Comp
-L power:+3V3 #PWR?
+L power:+3V3 #PWR0120
 U 1 1 614E43BC
 P 6650 5250
-F 0 "#PWR?" H 6650 5100 50  0001 C CNN
+F 0 "#PWR0120" H 6650 5100 50  0001 C CNN
 F 1 "+3V3" V 6665 5378 50  0000 L CNN
 F 2 "" H 6650 5250 50  0001 C CNN
@@
 	6650 5050 6900 5050
 $Comp
-L power:+3V3 #PWR?
+L power:+3V3 #PWR0121
 U 1 1 614F6F16
 P 8100 5250
-F 0 "#PWR?" H 8100 5100 50  0001 C CNN
+F 0 "#PWR0121" H 8100 5100 50  0001 C CNN
 F 1 "+3V3" V 8115 5378 50  0000 L CNN
 F 2 "" H 8100 5250 50  0001 C CNN
@@
 STLINK_SWDIO
 $Comp
-L power:GND #PWR?
+L power:GND #PWR0122
 U 1 1 61520E94
 P 8750 5050
-F 0 "#PWR?" H 8750 4800 50  0001 C CNN
+F 0 "#PWR0122" H 8750 4800 50  0001 C CNN
 F 1 "GND" V 8755 4922 50  0000 R CNN
 F 2 "" H 8750 5050 50  0001 C CNN
@@
 $EndComp
 $Comp
-L power:GND #PWR?
+L power:GND #PWR0123
 U 1 1 6155A083
 P 11050 2600
-F 0 "#PWR?" H 11050 2350 50  0001 C CNN
+F 0 "#PWR0123" H 11050 2350 50  0001 C CNN
 F 1 "GND" H 11055 2427 50  0000 C CNN
 F 2 "" H 11050 2600 50  0001 C CNN
@@
 	9650 2600 9350 2600
 $Comp
-L power:GND #PWR?
+L power:GND #PWR0124
 U 1 1 615676AA
 P 9350 2600
-F 0 "#PWR?" H 9350 2350 50  0001 C CNN
+F 0 "#PWR0124" H 9350 2350 50  0001 C CNN
 F 1 "GND" H 9355 2427 50  0000 C CNN
 F 2 "" H 9350 2600 50  0001 C CNN
@@
 	8550 6200 8550 6000
 $Comp
-L power:GND #PWR?
+L power:GND #PWR0125
 U 1 1 61630D6B
 P 8300 6300
-F 0 "#PWR?" H 8300 6050 50  0001 C CNN
+F 0 "#PWR0125" H 8300 6050 50  0001 C CNN
 F 1 "GND" H 8305 6127 50  0000 C CNN
 F 2 "" H 8300 6300 50  0001 C CNN
@@
 	8300 6200 8550 6200
 $Comp
-L power:VBUS #PWR?
+L power:VBUS #PWR0126
 U 1 1 6164474E
 P 10850 3050
-F 0 "#PWR?" H 10850 2900 50  0001 C CNN
+F 0 "#PWR0126" H 10850 2900 50  0001 C CNN
 F 1 "VBUS" H 10865 3223 50  0000 C CNN
 F 2 "" H 10850 3050 50  0001 C CNN
@@
 F 0 "R?" H 10909 2946 50  0000 L CNN
 F 1 "0R" H 10909 2855 50  0000 L CNN
-F 2 "" H 10850 2900 50  0001 C CNN
+F 2 "Resistor_SMD:R_0805_2012Metric_Pad1.20x1.40mm_HandSolder" H 10850 2900 50  0001 C CNN
 F 3 "~" H 10850 2900 50  0001 C CNN
 	1    10850 2900
@@
 	1300 4750 950  4750
 $Comp
-L power:GND #PWR?
+L power:GND #PWR0127
 U 1 1 616B826B
 P 1300 4900
-F 0 "#PWR?" H 1300 4650 50  0001 C CNN
+F 0 "#PWR0127" H 1300 4650 50  0001 C CNN
 F 1 "GND" H 1305 4727 50  0000 C CNN
 F 2 "" H 1300 4900 50  0001 C CNN

Commit message: PCB
PCB'ye geçildi. Boyutları düzeltilerek PCB'ye devam edilecek.
Parts:
- D7: renamed from D?; footprint SOT95P280X145-6N -> ESDA6V1BC6:SOT95P280X145-6N
- gave numbers to parts that had none: 42
- renumbered STLINK_CONN to STLINK_CONN1
Connections:
- net USB_DM renamed USB_N
- net USB_DP renamed USB_P
Other:
- moved on the sheet: R13
